File: SMC-80.sch (KiCad schematic (older format))
At the start: 8 parts, among them J1 RC80 Bus, J2 RC80 Expansion, SW1 Reset, U1 DS1813R-5+T&R

Commit message: Renamed to SMC-80
Parts:
- U1: symbol THS-80:DS1813R-5+T&R -> SMC-80:DS1813R-5+T&R
Changed lines of the file:
@@
 encoding utf-8
 Sheet 1 6
-Title "THS-80"
-Date "2019-08-15"
+Title "SMC-80"
+Date "2020-04-18"
 Rev "1.0"
 Comp "Hyiger Designs"
@@
 Connection ~ 5000 5600
 $Comp
-L THS-80:DS1813R-5+T&R U1
+L SMC-80:DS1813R-5+T&R U1
 U 1 1 5E47A0E9
 P 5100 5200

Commit message: trace routing
Connections:
- net labels added: A[0..13]
- net labels removed: A16, A17, A18, A[0..18]
- wire segments 181 -> 175
- no-connect marks 54 -> 60
Changed lines of the file:
@@
 	3350 3300 2950 3300
-Wire Wire Line
-	4250 4800 3850 4800
-Wire Wire Line
-	4250 4700 3850 4700
-Wire Wire Line
-	4250 4600 3850 4600
 Wire Wire Line
 	3850 5700 4250 5700
@@
 Text Label 3250 3300 2    50   ~ 0
 A15
-Text Label 4150 4800 2    50   ~ 0
-A16
-Text Label 4150 4700 2    50   ~ 0
-A17
-Text Label 4150 4600 2    50   ~ 0
-A18
 Text Label 3250 5900 2    50   ~ 0
 D0
@@
 	1350 3300 950  3300
 Wire Wire Line
-	2250 4800 1850 4800
-Wire Wire Line
-	2250 4700 1850 4700
-Wire Wire Line
-	2250 4600 1850 4600
-Wire Wire Line
 	1850 5700 2250 5700
 Wire Wire Line
@@
 Text Label 1250 3300 2    50   ~ 0
 A15
-Text Label 2150 4800 2    50   ~ 0
-A16
-Text Label 2150 4700 2    50   ~ 0
-A17
-Text Label 2150 4600 2    50   ~ 0
-A18
 Text Label 1250 5900 2    50   ~ 0
 D0
@@
 $EndSheet
 Text Label 9625 4050 0    50   ~ 0
-A[0..18]
+A[0..13]
 Wire Bus Line
 	10200 4050 9550 4050
@@
 NoConn ~ 1850 6000
 NoConn ~ 1850 5900
+NoConn ~ 3850 4800
+NoConn ~ 3850 4700
+NoConn ~ 3850 4600
+NoConn ~ 1850 4800
+NoConn ~ 1850 4700
+NoConn ~ 1850 4600
 $EndSCHEMATC

Commit message: Routing finished
Parts:
- removed JP1: Reset Ena, Connector_PinHeader_2.54mm:PinHeader_1x03_P2.54mm_Vertical, symbol Jumper:Jumper_3_Bridged12
- removed R1: 10K, Resistor_SMD:R_0603_1608Metric_Pad1.05x0.95mm_HandSolder, symbol Device:R_Small
- removed SW1: Reset, Button_Switch_SMD:SW_SPST_FSMSM, symbol Switch:SW_Push
- removed U1: DS1813R-5+T&R, Package_TO_SOT_SMD:SOT-23, symbol SMC-80:DS1813R-5+T&R
- added JP5: Reset Ena, Connector_PinHeader_2.54mm:PinHeader_1x03_P2.54mm_Vertical, symbol Jumper:Jumper_3_Bridged12
- added R21: 10K, Resistor_SMD:R_0603_1608Metric_Pad1.05x0.95mm_HandSolder, symbol Device:R_Small
- added SW3: Reset, Button_Switch_SMD:SW_SPST_FSMSM, symbol Switch:SW_Push
- added U14: DS1813R-5+T&R, Package_TO_SOT_SMD:SOT-23, symbol SMC-80:DS1813R-5+T&R
Connections:
- net labels added: A[0..15]
- net labels removed: A[0..13]
Other:
- moved on the sheet: C1, J1, J2, RN1

Commit message: remove old files, added jtag pullup
Parts:
- renumbered JP5 to JP1, R21 to R1, SW3 to SW1, U14 to U1
Changed lines of the file:
@@
 	4250 2600 3850 2600
 $Comp
-L power:GND #PWR03
+L power:GND #PWR05
 U 1 1 616B6DD8
 P 2400 2650
-AR Path="/616B6DD8" Ref="#PWR03"  Part="1"
+AR Path="/616B6DD8" Ref="#PWR05"  Part="1"
 AR Path="/5CB63856/616B6DD8" Ref="#PWR?"  Part="1"
 AR Path="/5CB5AB00/5CB63856/616B6DD8" Ref="#PWR?"  Part="1"
-F 0 "#PWR03" H 2400 2400 50  0001 C CNN
+F 0 "#PWR05" H 2400 2400 50  0001 C CNN
 F 1 "GND" H 2405 2477 50  0000 C CNN
 F 2 "" H 2400 2650 50  0001 C CNN
@@
 	5850 4100 5850 4200
 $Comp
-L power:VCC #PWR04
+L power:VCC #PWR07
 U 1 1 5E47A107
 P 5850 4100
-F 0 "#PWR04" H 5850 3950 50  0001 C CNN
+F 0 "#PWR07" H 5850 3950 50  0001 C CNN
 F 1 "VCC" H 5867 4273 50  0000 C CNN
 F 2 "" H 5850 4100 50  0001 C CNN
@@
 Connection ~ 1550 6750
 $Comp
-L SMC-80:DS1813R-5+T&R U14
+L SMC-80:DS1813R-5+T&R U1
 U 1 1 5EFC5345
 P 1650 6350
-AR Path="/5EFC5345" Ref="U14"  Part="1"
+AR Path="/5EFC5345" Ref="U1"  Part="1"
 AR Path="/5D6224DC/5EFC5345" Ref="U?"  Part="1"
 AR Path="/5F7E53CF/5EFC5345" Ref="U?"  Part="1"
-F 0 "U14" H 1420 6396 50  0000 R CNN
+F 0 "U1" H 1420 6396 50  0000 R CNN
 F 1 "DS1813R-5+T&R" H 2300 6700 50  0000 R CNN
 F 2 "Package_TO_SOT_SMD:SOT-23" H 1250 6500 50  0001 C CNN
@@
 $EndComp
 $Comp
-L Switch:SW_Push SW3
+L Switch:SW_Push SW1
 U 1 1 5EFC534B
 P 2150 6550
-AR Path="/5EFC534B" Ref="SW3"  Part="1"
+AR Path="/5EFC534B" Ref="SW1"  Part="1"
 AR Path="/5D6224DC/5EFC534B" Ref="SW?"  Part="1"
 AR Path="/5F7E53CF/5EFC534B" Ref="SW?"  Part="1"
-F 0 "SW3" V 2104 6698 50  0000 L CNN
+F 0 "SW1" V 2104 6698 50  0000 L CNN
 F 1 "Reset" V 2195 6698 50  0000 L CNN
 F 2 "Button_Switch_SMD:SW_SPST_FSMSM" H 2150 6750 50  0001 C CNN
@@
 	2150 6350 2600 6350
 $Comp
-L power:GND #PWR0101
+L power:GND #PWR04
 U 1 1 5EFC5352
 P 1550 6850
-AR Path="/5EFC5352" Ref="#PWR0101"  Part="1"
+AR Path="/5EFC5352" Ref="#PWR04"  Part="1"
 AR Path="/5CB63856/5EFC5352" Ref="#PWR?"  Part="1"
 AR Path="/5CB5AB00/5CB63856/5EFC5352" Ref="#PWR?"  Part="1"
@@
 AR Path="/5D6224DC/5EFC5352" Ref="#PWR?"  Part="1"
 AR Path="/5F7E53CF/5EFC5352" Ref="#PWR?"  Part="1"
-F 0 "#PWR0101" H 1550 6600 50  0001 C CNN
+F 0 "#PWR04" H 1550 6600 50  0001 C CNN
 F 1 "GND" H 1554 6708 50  0000 C CNN
 F 2 "" H 1550 6850 50  0001 C CNN
@@
 	1550 6750 1550 6850
 $Comp
-L power:VCC #PWR0102
+L power:VCC #PWR03
 U 1 1 5EFC5359
 P 1550 5950
-AR Path="/5EFC5359" Ref="#PWR0102"  Part="1"
+AR Path="/5EFC5359" Ref="#PWR03"  Part="1"
 AR Path="/5F7E53CF/5EFC5359" Ref="#PWR?"  Part="1"
-F 0 "#PWR0102" H 1550 5800 50  0001 C CNN
+F 0 "#PWR03" H 1550 5800 50  0001 C CNN
 F 1 "VCC" H 1567 6123 50  0000 C CNN
 F 2 "" H 1550 5950 50  0001 C CNN
@@
 $EndComp
 $Comp
-L Jumper:Jumper_3_Bridged12 JP5
+L Jumper:Jumper_3_Bridged12 JP1
 U 1 1 5EFC535F
 P 2850 6350
-AR Path="/5EFC535F" Ref="JP5"  Part="1"
+AR Path="/5EFC535F" Ref="JP1"  Part="1"
 AR Path="/5F7E53CF/5EFC535F" Ref="JP?"  Part="1"
-F 0 "JP5" H 2850 6554 50  0000 C CNN
+F 0 "JP1" H 2850 6554 50  0000 C CNN
 F 1 "Reset Ena" H 2850 6463 50  0000 C CNN
 F 2 "Connector_PinHeader_2.54mm:PinHeader_1x03_P2.54mm_Vertical" H 2850 6350 50  0001 C CNN
@@
 	3100 6350 3550 6350
 $Comp
-L Device:R_Small R21
+L Device:R_Small R1
 U 1 1 5EFC5368
 P 3550 6150
-AR Path="/5EFC5368" Ref="R21"  Part="1"
+AR Path="/5EFC5368" Ref="R1"  Part="1"
 AR Path="/5D6224DC/5EFC5368" Ref="R?"  Part="1"
 AR Path="/5F7E53CF/5EFC5368" Ref="R?"  Part="1"
-F 0 "R21" V 3475 6075 50  0000 L CNN
+F 0 "R1" V 3475 6075 50  0000 L CNN
 F 1 "10K" V 3550 6100 32  0000 L CNN
 F 2 "Resistor_SMD:R_0603_1608Metric_Pad1.05x0.95mm_HandSolder" H 3550 6150 50  0001 C CNN
@@
 $EndComp
 $Comp
-L power:VCC #PWR0103
+L power:VCC #PWR06
 U 1 1 5EFC536E
 P 3550 6050
-AR Path="/5EFC536E" Ref="#PWR0103"  Part="1"
+AR Path="/5EFC536E" Ref="#PWR06"  Part="1"
 AR Path="/5F7E53CF/5EFC536E" Ref="#PWR?"  Part="1"
-F 0 "#PWR0103" H 3550 5900 50  0001 C CNN
+F 0 "#PWR06" H 3550 5900 50  0001 C CNN
 F 1 "VCC" H 3567 6223 50  0000 C CNN
 F 2 "" H 3550 6050 50  0001 C CNN
