File: cpu_ram_rom.sch (KiCad schematic (older format))
At the start: 9 parts, among them U10 Z84C0010AEG, U11 SST39SF040, U9 AS6C4008A-55ZIN

Commit message: Renamed to SMC-80
Parts:
- U10: symbol THS-80:Z84C0010AEG -> SMC-80:Z84C0010AEG
- U9: symbol THS-80-rescue:AS6C4008A-55ZIN-Memory_RAM -> SMC-80-rescue:AS6C4008A-55ZIN-Memory_RAM
Changed lines of the file:
@@
 $EndComp
 $Comp
-L THS-80:Z84C0010AEG U10
+L SMC-80:Z84C0010AEG U10
 U 1 1 5F309FF5
 P 3900 5750
@@
 $EndComp
 $Comp
-L THS-80-rescue:AS6C4008A-55ZIN-Memory_RAM U9
+L SMC-80-rescue:AS6C4008A-55ZIN-Memory_RAM U9
 U 1 1 5DA31E6C
 P 3750 1900

Commit message: trace routing
Changed lines of the file:
@@
 	5250 6950 5350 7050
 Text HLabel 5350 5350 2    50   Output ~ 0
-A[0..18]
+A[0..15]
 Text HLabel 5350 6650 2    50   3State ~ 0
 D[0..7]
@@
 	2700 2500 2600 2600
 Text HLabel 2600 1750 0    50   Input ~ 0
-A[0..18]
+A[0..15]
 Entry Wire Line
 	10750 800  10850 900
@@
 ~RD
 Text HLabel 8350 1700 0    50   Input ~ 0
-A[0..18]
+A[0..15]
 Entry Wire Line
 	8450 2100 8350 2200

Commit message: Routing finished
Parts:
- renumbered C24 to C21, C25 to C22, C26 to C23, JP5 to JP4, R17 to R16, R18 to R17, U9 to U7, U10 to U8, U11 to U9
Other:
- moved on the sheet: C21, C22, C23
Changed lines of the file:
@@
 $Descr A4 11693 8268
 encoding utf-8
-Sheet 5 6
+Sheet 4 5
 Title ""
 Date ""
@@
 AR Path="/5CFABACD/5D90DF01" Ref="#PWR?"  Part="1"
 AR Path="/5CF9C1ED/5D90DF01" Ref="#PWR?"  Part="1"
-AR Path="/5D6224DC/5D90DF01" Ref="#PWR074"  Part="1"
-F 0 "#PWR074" H 3750 2750 50  0001 C CNN
+AR Path="/5D6224DC/5D90DF01" Ref="#PWR066"  Part="1"
+F 0 "#PWR066" H 3750 2750 50  0001 C CNN
 F 1 "GND" H 3755 2827 50  0000 C CNN
 F 2 "" H 3750 3000 50  0001 C CNN
@@
 $EndComp
 $Comp
-L SMC-80:Z84C0010AEG U10
+L SMC-80:Z84C0010AEG U8
 U 1 1 5F309FF5
 P 3900 5750
-F 0 "U10" H 3350 7200 50  0000 C CNN
+F 0 "U8" H 3350 7200 50  0000 C CNN
 F 1 "Z84C0010AEG" H 3900 5750 50  0000 C CNN
 F 2 "Package_QFP:LQFP-44_10x10mm_P0.8mm" H 950 6750 50  0001 L CNN
@@
 AR Path="/5CFABACD/5F33A976" Ref="#PWR?"  Part="1"
 AR Path="/5CF9C1ED/5F33A976" Ref="#PWR?"  Part="1"
-AR Path="/5D6224DC/5F33A976" Ref="#PWR076"  Part="1"
-F 0 "#PWR076" H 3900 7050 50  0001 C CNN
+AR Path="/5D6224DC/5F33A976" Ref="#PWR068"  Part="1"
+F 0 "#PWR068" H 3900 7050 50  0001 C CNN
 F 1 "GND" H 3905 7127 50  0000 C CNN
 F 2 "" H 3900 7300 50  0001 C CNN
@@
 L power:GND #PWR?
 U 1 1 5FC53564
-P 6850 5850
+P 8150 5600
 AR Path="/5D70CA34/5FC53564" Ref="#PWR?"  Part="1"
-AR Path="/5D6224DC/5FC53564" Ref="#PWR079"  Part="1"
-F 0 "#PWR079" H 6850 5600 50  0001 C CNN
-F 1 "GND" H 6855 5677 50  0000 C CNN
-F 2 "" H 6850 5850 50  0001 C CNN
-F 3 "" H 6850 5850 50  0001 C CNN
-	1    6850 5850
-	1    0    0    -1
-$EndComp
-$Comp
-L Device:R_Small R18
+AR Path="/5D6224DC/5FC53564" Ref="#PWR073"  Part="1"
+F 0 "#PWR073" H 8150 5350 50  0001 C CNN
+F 1 "GND" H 8155 5427 50  0000 C CNN
+F 2 "" H 8150 5600 50  0001 C CNN
+F 3 "" H 8150 5600 50  0001 C CNN
+	1    8150 5600
+	1    0    0    -1
+$EndComp
+$Comp
+L Device:R_Small R17
 U 1 1 5D959555
 P 7550 2900
-F 0 "R18" H 7609 2946 50  0000 L CNN
+F 0 "R17" H 7609 2946 50  0000 L CNN
 F 1 "10K" H 7609 2855 50  0000 L CNN
 F 2 "Resistor_SMD:R_0603_1608Metric_Pad1.05x0.95mm_HandSolder" H 7550 2900 50  0001 C CNN
@@
 $EndComp
 $Comp
-L Device:R_Small R17
+L Device:R_Small R16
 U 1 1 5D966170
 P 5700 1900
-F 0 "R17" H 5759 1946 50  0000 L CNN
+F 0 "R16" H 5759 1946 50  0000 L CNN
 F 1 "10K" H 5759 1855 50  0000 L CNN
 F 2 "Resistor_SMD:R_0603_1608Metric_Pad1.05x0.95mm_HandSolder" H 5700 1900 50  0001 C CNN
@@
 Flash/ROM
 $Comp
-L Memory_Flash:SST39SF040 U11
+L Memory_Flash:SST39SF040 U9
 U 1 1 5D653323
 P 9600 2000
-F 0 "U11" H 9250 3300 50  0000 C CNN
+F 0 "U9" H 9250 3300 50  0000 C CNN
 F 1 "SST39SF040" H 9650 2050 50  0000 C CNN
 F 2 "Package_LCC:PLCC-32_11.4x14.0mm_P1.27mm" H 9600 2300 50  0001 C CNN
@@
 Connection ~ 7550 3000
 $Comp
-L Device:C_Small C24
+L Device:C_Small C21
 U 1 1 5F181CA3
-P 6500 5700
-F 0 "C24" H 6592 5746 50  0000 L CNN
-F 1 "100nF" H 6592 5655 50  0000 L CNN
-F 2 "Capacitor_SMD:C_0603_1608Metric_Pad1.05x0.95mm_HandSolder" H 6500 5700 50  0001 C CNN
-F 3 "~" H 6500 5700 50  0001 C CNN
-	1    6500 5700
-	1    0    0    -1
-$EndComp
-$Comp
-L Device:C_Small C25
+P 7800 5450
+F 0 "C21" H 7892 5496 50  0000 L CNN
+F 1 "100nF" H 7892 5405 50  0000 L CNN
+F 2 "Capacitor_SMD:C_0603_1608Metric_Pad1.05x0.95mm_HandSolder" H 7800 5450 50  0001 C CNN
+F 3 "~" H 7800 5450 50  0001 C CNN
+	1    7800 5450
+	1    0    0    -1
+$EndComp
+$Comp
+L Device:C_Small C22
 U 1 1 5F182ACB
-P 6850 5700
-F 0 "C25" H 6942 5746 50  0000 L CNN
-F 1 "100nF" H 6942 5655 50  0000 L CNN
-F 2 "Capacitor_SMD:C_0603_1608Metric_Pad1.05x0.95mm_HandSolder" H 6850 5700 50  0001 C CNN
-F 3 "~" H 6850 5700 50  0001 C CNN
-	1    6850 5700
-	1    0    0    -1
-$EndComp
-$Comp
-L Device:C_Small C26
+P 8150 5450
+F 0 "C22" H 8242 5496 50  0000 L CNN
+F 1 "100nF" H 8242 5405 50  0000 L CNN
+F 2 "Capacitor_SMD:C_0603_1608Metric_Pad1.05x0.95mm_HandSolder" H 8150 5450 50  0001 C CNN
+F 3 "~" H 8150 5450 50  0001 C CNN
+	1    8150 5450
+	1    0    0    -1
+$EndComp
+$Comp
+L Device:C_Small C23
 U 1 1 5F189729
-P 7250 5700
-F 0 "C26" H 7342 5746 50  0000 L CNN
-F 1 "100nF" H 7342 5655 50  0000 L CNN
-F 2 "Capacitor_SMD:C_0603_1608Metric_Pad1.05x0.95mm_HandSolder" H 7250 5700 50  0001 C CNN
-F 3 "~" H 7250 5700 50  0001 C CNN
-	1    7250 5700
-	1    0    0    -1
-$EndComp
-Wire Wire Line
-	6500 5600 6500 5550
-Wire Wire Line
-	6500 5550 6850 5550
-Wire Wire Line
-	7250 5550 7250 5600
-Wire Wire Line
-	6850 5600 6850 5550
-Connection ~ 6850 5550
-Wire Wire Line
-	6850 5550 7250 5550
-Wire Wire Line
-	6500 5800 6500 5850
-Wire Wire Line
-	6500 5850 6850 5850
-Wire Wire Line
-	7250 5850 7250 5800
-Wire Wire Line
-	6850 5800 6850 5850
-Connection ~ 6850 5850
-Wire Wire Line
-	6850 5850 7250 5850
+P 8550 5450
+F 0 "C23" H 8642 5496 50  0000 L CNN
+F 1 "100nF" H 8642 5405 50  0000 L CNN
+F 2 "Capacitor_SMD:C_0603_1608Metric_Pad1.05x0.95mm_HandSolder" H 8550 5450 50  0001 C CNN
+F 3 "~" H 8550 5450 50  0001 C CNN
+	1    8550 5450
+	1    0    0    -1
+$EndComp
+Wire Wire Line
+	7800 5350 7800 5300
+Wire Wire Line
+	7800 5300 8150 5300
+Wire Wire Line
+	8550 5300 8550 5350
+Wire Wire Line
+	8150 5350 8150 5300
+Connection ~ 8150 5300
+Wire Wire Line
+	8150 5300 8550 5300
+Wire Wire Line
+	7800 5550 7800 5600
+Wire Wire Line
+	7800 5600 8150 5600
+Wire Wire Line
+	8550 5600 8550 5550
+Wire Wire Line
+	8150 5550 8150 5600
+Connection ~ 8150 5600
+Wire Wire Line
+	8150 5600 8550 5600
 Wire Wire Line
 	7550 3000 9000 3000
@@
 P 7550 2800
 AR Path="/5DC9BD0A" Ref="#PWR?"  Part="1"
-AR Path="/5D6224DC/5DC9BD0A" Ref="#PWR081"  Part="1"
-F 0 "#PWR081" H 7550 2650 50  0001 C CNN
+AR Path="/5D6224DC/5DC9BD0A" Ref="#PWR071"  Part="1"
+F 0 "#PWR071" H 7550 2650 50  0001 C CNN
 F 1 "VCC" H 7567 2973 50  0000 C CNN
 F 2 "" H 7550 2800 50  0001 C CNN
@@
 P 7550 1950
 AR Path="/5DCA243D" Ref="#PWR?"  Part="1"
-AR Path="/5D6224DC/5DCA243D" Ref="#PWR080"  Part="1"
-F 0 "#PWR080" H 7550 1800 50  0001 C CNN
+AR Path="/5D6224DC/5DCA243D" Ref="#PWR070"  Part="1"
+F 0 "#PWR070" H 7550 1800 50  0001 C CNN
 F 1 "VCC" H 7567 2123 50  0000 C CNN
 F 2 "" H 7550 1950 50  0001 C CNN
@@
 P 3750 800
 AR Path="/5DCD0880" Ref="#PWR?"  Part="1"
-AR Path="/5D6224DC/5DCD0880" Ref="#PWR073"  Part="1"
-F 0 "#PWR073" H 3750 650 50  0001 C CNN
+AR Path="/5D6224DC/5DCD0880" Ref="#PWR065"  Part="1"
+F 0 "#PWR065" H 3750 650 50  0001 C CNN
 F 1 "VCC" H 3767 973 50  0000 C CNN
 F 2 "" H 3750 800 50  0001 C CNN
@@
 P 5700 1800
 AR Path="/5DCDDE0E" Ref="#PWR?"  Part="1"
-AR Path="/5D6224DC/5DCDDE0E" Ref="#PWR077"  Part="1"
-F 0 "#PWR077" H 5700 1650 50  0001 C CNN
+AR Path="/5D6224DC/5DCDDE0E" Ref="#PWR069"  Part="1"
+F 0 "#PWR069" H 5700 1650 50  0001 C CNN
 F 1 "VCC" H 5717 1973 50  0000 C CNN
 F 2 "" H 5700 1800 50  0001 C CNN
@@
 P 3900 4200
 AR Path="/5DCEC440" Ref="#PWR?"  Part="1"
-AR Path="/5D6224DC/5DCEC440" Ref="#PWR075"  Part="1"
-F 0 "#PWR075" H 3900 4050 50  0001 C CNN
+AR Path="/5D6224DC/5DCEC440" Ref="#PWR067"  Part="1"
+F 0 "#PWR067" H 3900 4050 50  0001 C CNN
 F 1 "VCC" H 3917 4373 50  0000 C CNN
 F 2 "" H 3900 4200 50  0001 C CNN
@@
 P 9600 700
 AR Path="/5DCF306D" Ref="#PWR?"  Part="1"
-AR Path="/5D6224DC/5DCF306D" Ref="#PWR082"  Part="1"
-F 0 "#PWR082" H 9600 550 50  0001 C CNN
+AR Path="/5D6224DC/5DCF306D" Ref="#PWR074"  Part="1"
+F 0 "#PWR074" H 9600 550 50  0001 C CNN
 F 1 "VCC" H 9617 873 50  0000 C CNN
 F 2 "" H 9600 700 50  0001 C CNN
@@
 L power:VCC #PWR?
 U 1 1 5DD0030A
-P 6850 5550
+P 8150 5300
 AR Path="/5DD0030A" Ref="#PWR?"  Part="1"
-AR Path="/5D6224DC/5DD0030A" Ref="#PWR078"  Part="1"
-F 0 "#PWR078" H 6850 5400 50  0001 C CNN
-F 1 "VCC" H 6867 5723 50  0000 C CNN
-F 2 "" H 6850 5550 50  0001 C CNN
-F 3 "" H 6850 5550 50  0001 C CNN
-	1    6850 5550
-	1    0    0    -1
-$EndComp
-$Comp
-L SMC-80-rescue:AS6C4008A-55ZIN-Memory_RAM U9
+AR Path="/5D6224DC/5DD0030A" Ref="#PWR072"  Part="1"
+F 0 "#PWR072" H 8150 5150 50  0001 C CNN
+F 1 "VCC" H 8167 5473 50  0000 C CNN
+F 2 "" H 8150 5300 50  0001 C CNN
+F 3 "" H 8150 5300 50  0001 C CNN
+	1    8150 5300
+	1    0    0    -1
+$EndComp
+$Comp
+L SMC-80-rescue:AS6C4008A-55ZIN-Memory_RAM U7
 U 1 1 5DA31E6C
 P 3750 1900
-F 0 "U9" H 3400 3000 50  0000 C CNN
+F 0 "U7" H 3400 3000 50  0000 C CNN
 F 1 "AS6C4008A-55ZIN" H 4200 3000 50  0000 C CNN
 F 2 "Package_SO:TSOP-II-32_21.0x10.2mm_P1.27mm" H 3750 2000 50  0001 C CNN
@@
 P 7550 2300
 AR Path="/5EA41998" Ref="JP?"  Part="1"
-AR Path="/5D6224DC/5EA41998" Ref="JP5"  Part="1"
-F 0 "JP5" V 7550 2504 50  0000 C CNN
+AR Path="/5D6224DC/5EA41998" Ref="JP4"  Part="1"
+F 0 "JP4" V 7550 2504 50  0000 C CNN
 F 1 "WR Ena" V 7650 2500 50  0000 C CNN
 F 2 "Connector_PinHeader_2.54mm:PinHeader_1x03_P2.54mm_Vertical" H 7550 2300 50  0001 C CNN

Commit message: remove old files, added jtag pullup
Parts:
- renumbered JP4 to JP5, R16 to R18, R17 to R19, U9 to U10, U7 to U8, U8 to U9
Changed lines of the file:
@@
 AR Path="/5CFABACD/5D90DF01" Ref="#PWR?"  Part="1"
 AR Path="/5CF9C1ED/5D90DF01" Ref="#PWR?"  Part="1"
-AR Path="/5D6224DC/5D90DF01" Ref="#PWR066"  Part="1"
-F 0 "#PWR066" H 3750 2750 50  0001 C CNN
+AR Path="/5D6224DC/5D90DF01" Ref="#PWR069"  Part="1"
+F 0 "#PWR069" H 3750 2750 50  0001 C CNN
 F 1 "GND" H 3755 2827 50  0000 C CNN
 F 2 "" H 3750 3000 50  0001 C CNN
@@
 $EndComp
 $Comp
-L SMC-80:Z84C0010AEG U8
+L SMC-80:Z84C0010AEG U9
 U 1 1 5F309FF5
 P 3900 5750
-F 0 "U8" H 3350 7200 50  0000 C CNN
+F 0 "U9" H 3350 7200 50  0000 C CNN
 F 1 "Z84C0010AEG" H 3900 5750 50  0000 C CNN
 F 2 "Package_QFP:LQFP-44_10x10mm_P0.8mm" H 950 6750 50  0001 L CNN
@@
 AR Path="/5CFABACD/5F33A976" Ref="#PWR?"  Part="1"
 AR Path="/5CF9C1ED/5F33A976" Ref="#PWR?"  Part="1"
-AR Path="/5D6224DC/5F33A976" Ref="#PWR068"  Part="1"
-F 0 "#PWR068" H 3900 7050 50  0001 C CNN
+AR Path="/5D6224DC/5F33A976" Ref="#PWR071"  Part="1"
+F 0 "#PWR071" H 3900 7050 50  0001 C CNN
 F 1 "GND" H 3905 7127 50  0000 C CNN
 F 2 "" H 3900 7300 50  0001 C CNN
@@
 P 8150 5600
 AR Path="/5D70CA34/5FC53564" Ref="#PWR?"  Part="1"
-AR Path="/5D6224DC/5FC53564" Ref="#PWR073"  Part="1"
-F 0 "#PWR073" H 8150 5350 50  0001 C CNN
+AR Path="/5D6224DC/5FC53564" Ref="#PWR076"  Part="1"
+F 0 "#PWR076" H 8150 5350 50  0001 C CNN
 F 1 "GND" H 8155 5427 50  0000 C CNN
 F 2 "" H 8150 5600 50  0001 C CNN
@@
 $EndComp
 $Comp
-L Device:R_Small R17
+L Device:R_Small R19
 U 1 1 5D959555
 P 7550 2900
-F 0 "R17" H 7609 2946 50  0000 L CNN
+F 0 "R19" H 7609 2946 50  0000 L CNN
 F 1 "10K" H 7609 2855 50  0000 L CNN
 F 2 "Resistor_SMD:R_0603_1608Metric_Pad1.05x0.95mm_HandSolder" H 7550 2900 50  0001 C CNN
@@
 $EndComp
 $Comp
-L Device:R_Small R16
+L Device:R_Small R18
 U 1 1 5D966170
 P 5700 1900
-F 0 "R16" H 5759 1946 50  0000 L CNN
+F 0 "R18" H 5759 1946 50  0000 L CNN
 F 1 "10K" H 5759 1855 50  0000 L CNN
 F 2 "Resistor_SMD:R_0603_1608Metric_Pad1.05x0.95mm_HandSolder" H 5700 1900 50  0001 C CNN
@@
 Flash/ROM
 $Comp
-L Memory_Flash:SST39SF040 U9
+L Memory_Flash:SST39SF040 U10
 U 1 1 5D653323
 P 9600 2000
-F 0 "U9" H 9250 3300 50  0000 C CNN
+F 0 "U10" H 9250 3300 50  0000 C CNN
 F 1 "SST39SF040" H 9650 2050 50  0000 C CNN
 F 2 "Package_LCC:PLCC-32_11.4x14.0mm_P1.27mm" H 9600 2300 50  0001 C CNN
@@
 P 7550 2800
 AR Path="/5DC9BD0A" Ref="#PWR?"  Part="1"
-AR Path="/5D6224DC/5DC9BD0A" Ref="#PWR071"  Part="1"
-F 0 "#PWR071" H 7550 2650 50  0001 C CNN
+AR Path="/5D6224DC/5DC9BD0A" Ref="#PWR074"  Part="1"
+F 0 "#PWR074" H 7550 2650 50  0001 C CNN
 F 1 "VCC" H 7567 2973 50  0000 C CNN
 F 2 "" H 7550 2800 50  0001 C CNN
@@
 P 7550 1950
 AR Path="/5DCA243D" Ref="#PWR?"  Part="1"
-AR Path="/5D6224DC/5DCA243D" Ref="#PWR070"  Part="1"
-F 0 "#PWR070" H 7550 1800 50  0001 C CNN
+AR Path="/5D6224DC/5DCA243D" Ref="#PWR073"  Part="1"
+F 0 "#PWR073" H 7550 1800 50  0001 C CNN
 F 1 "VCC" H 7567 2123 50  0000 C CNN
 F 2 "" H 7550 1950 50  0001 C CNN
@@
 P 3750 800
 AR Path="/5DCD0880" Ref="#PWR?"  Part="1"
-AR Path="/5D6224DC/5DCD0880" Ref="#PWR065"  Part="1"
-F 0 "#PWR065" H 3750 650 50  0001 C CNN
+AR Path="/5D6224DC/5DCD0880" Ref="#PWR068"  Part="1"
+F 0 "#PWR068" H 3750 650 50  0001 C CNN
 F 1 "VCC" H 3767 973 50  0000 C CNN
 F 2 "" H 3750 800 50  0001 C CNN
@@
 P 5700 1800
 AR Path="/5DCDDE0E" Ref="#PWR?"  Part="1"
-AR Path="/5D6224DC/5DCDDE0E" Ref="#PWR069"  Part="1"
-F 0 "#PWR069" H 5700 1650 50  0001 C CNN
+AR Path="/5D6224DC/5DCDDE0E" Ref="#PWR072"  Part="1"
+F 0 "#PWR072" H 5700 1650 50  0001 C CNN
 F 1 "VCC" H 5717 1973 50  0000 C CNN
 F 2 "" H 5700 1800 50  0001 C CNN
@@
 P 3900 4200
 AR Path="/5DCEC440" Ref="#PWR?"  Part="1"
-AR Path="/5D6224DC/5DCEC440" Ref="#PWR067"  Part="1"
-F 0 "#PWR067" H 3900 4050 50  0001 C CNN
+AR Path="/5D6224DC/5DCEC440" Ref="#PWR070"  Part="1"
+F 0 "#PWR070" H 3900 4050 50  0001 C CNN
 F 1 "VCC" H 3917 4373 50  0000 C CNN
 F 2 "" H 3900 4200 50  0001 C CNN
@@
 P 9600 700
 AR Path="/5DCF306D" Ref="#PWR?"  Part="1"
-AR Path="/5D6224DC/5DCF306D" Ref="#PWR074"  Part="1"
-F 0 "#PWR074" H 9600 550 50  0001 C CNN
+AR Path="/5D6224DC/5DCF306D" Ref="#PWR077"  Part="1"
+F 0 "#PWR077" H 9600 550 50  0001 C CNN
 F 1 "VCC" H 9617 873 50  0000 C CNN
 F 2 "" H 9600 700 50  0001 C CNN
@@
 P 8150 5300
 AR Path="/5DD0030A" Ref="#PWR?"  Part="1"
-AR Path="/5D6224DC/5DD0030A" Ref="#PWR072"  Part="1"
-F 0 "#PWR072" H 8150 5150 50  0001 C CNN
+AR Path="/5D6224DC/5DD0030A" Ref="#PWR075"  Part="1"
+F 0 "#PWR075" H 8150 5150 50  0001 C CNN
 F 1 "VCC" H 8167 5473 50  0000 C CNN
 F 2 "" H 8150 5300 50  0001 C CNN
@@
 $EndComp
 $Comp
-L SMC-80-rescue:AS6C4008A-55ZIN-Memory_RAM U7
+L SMC-80-rescue:AS6C4008A-55ZIN-Memory_RAM U8
 U 1 1 5DA31E6C
 P 3750 1900
-F 0 "U7" H 3400 3000 50  0000 C CNN
+F 0 "U8" H 3400 3000 50  0000 C CNN
 F 1 "AS6C4008A-55ZIN" H 4200 3000 50  0000 C CNN
 F 2 "Package_SO:TSOP-II-32_21.0x10.2mm_P1.27mm" H 3750 2000 50  0001 C CNN
@@
 P 7550 2300
 AR Path="/5EA41998" Ref="JP?"  Part="1"
-AR Path="/5D6224DC/5EA41998" Ref="JP4"  Part="1"
-F 0 "JP4" V 7550 2504 50  0000 C CNN
+AR Path="/5D6224DC/5EA41998" Ref="JP5"  Part="1"
+F 0 "JP5" V 7550 2504 50  0000 C CNN
 F 1 "WR Ena" V 7650 2500 50  0000 C CNN
 F 2 "Connector_PinHeader_2.54mm:PinHeader_1x03_P2.54mm_Vertical" H 7550 2300 50  0001 C CNN
